Commit message: fixed rviz2 model and wheel slipping problem

File: ackermancar_description/urdf/hunter.urdf (robot description, URDF)
Before this commit: robot Argus_Hunter_2, 18 links, 17 joints
Links:
- link base_link: geometry collision mesh filename=package://ackermancar_description/meshes/visual/chassis_and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; visual mesh filename=$(find ackermancar_description)/meshes/visual/chassis_and_f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

File: ackermancar_description/urdf/hunter.urdf.xacro (robot description, xacro)
@@ -4,5 +4,5 @@
      For more information, please see http://wiki.ros.org/sw_urdf_exporter -->
 <robot name="Argus_Hunter_2" xmlns:xacro="http://www.ros.org/wiki/xacro">
-  <xacro:property name="VISUAL_DIR" value="/home/youngricky/graduation_project_ws/src/ackermancar_description/meshes/visual"/>
+  <xacro:property name="VISUAL_DIR" value="$(find ackermancar_description)/meshes/visual"/>
   <xacro:property name="wheel_width" value="0.14"/>
   <xacro:property name="wheel_radius" value="0.165"/>
@@ -13,5 +13,5 @@
           xyz="0 0.0016115 0"
           rpy="0 0 0" />
-        <mass value="4.0" />
+        <mass value="5" />
         <inertia
           ixx="0.06368"
@@ -89,5 +89,5 @@
       <parent link="base_link" />
       <child link="${prefix}_steering_link" />
-      <dynamics damping="0.5" friction="0.01"/>
+      <dynamics damping="0.8" friction="0.1"/>
       <axis xyz="0 0 1" />
       <limit lower="-0.575" upper="0.575" effort="1000" velocity="100"/>
@@ -99,5 +99,5 @@
       <parent link="front_${prefix}_steering_link" />
       <child link="front_${prefix}_wheel" />
-      <dynamics damping="0.1" friction="0.1"/>
+      <dynamics damping="0.5" friction="0.5"/>
       <axis xyz="0 ${yaxis} 0" />
       <limit effort="1000.0" velocity="100"/>
@@ -109,5 +109,5 @@
       <parent link="base_link" />
       <child link="rear_${prefix}_wheel" />
-      <dynamics damping="0.1" friction="0.1"/>
+      <dynamics damping="0.5" friction="0.5"/>
       <axis xyz="0 ${yaxis} 0" />
       <limit effort="1000.0" velocity="500.0"/>

Commit message: seperate hunter.urdf.xacro into multiple files and change tire args

File: ackermancar_description/urdf/hunter.urdf (robot description, URDF)
Before this commit: robot Argus_Hunter_2, 18 links, 17 joints
Links:
- link base_link: geometry collision mesh filename=package://ackermancar_description/meshes/visual/chassis_and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; visual mesh filename=package://ackermancar_description/meshes/visual/chassis_and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

File: ackermancar_description/urdf/hunter.urdf.xacro (robot description, xacro)
@@ -402,13 +402,13 @@
     <material>Gazebo/White</material>
   </gazebo>
-  <xacro:gazebo_wheel prefix="front_left" mu1="1.0" mu2="1.0" kp="1e8" kd="1.0"/>
-  <xacro:gazebo_wheel prefix="front_right" mu1="1.0" mu2="1.0" kp="1e8" kd="1.0"/>
-  <xacro:gazebo_wheel prefix="rear_left" mu1="1.0" mu2="1.0" kp="1e8" kd="1.0"/>
-  <xacro:gazebo_wheel prefix="rear_right" mu1="1.0" mu2="1.0" kp="1e8" kd="1.0"/>
+  <xacro:gazebo_wheel prefix="front_left" mu1="5.0" mu2="5.0" kp="1e8" kd="1.0"/>
+  <xacro:gazebo_wheel prefix="front_right" mu1="5.0" mu2="5.0" kp="1e8" kd="1.0"/>
+  <xacro:gazebo_wheel prefix="rear_left" mu1="5.0" mu2="5.0" kp="1e8" kd="1.0"/>
+  <xacro:gazebo_wheel prefix="rear_right" mu1="5.0" mu2="5.0" kp="1e8" kd="1.0"/>
   <!-- ackmann driver model -->
   <gazebo>
     <plugin name="gazebo_ros_ackermann_drive" filename="libgazebo_ros_ackermann_drive.so">
       <ros>
-        <namespace>/orbbec_hunter2</namespace>
+        <namespace>/orbbec_hunter</namespace>
         <remapping> cmd_vel:=cmd_vel </remapping>
         <remapping> odom:=odom </remapping>
