Commit message: fix transform between footprint and baselink

File: ackermancar_description/urdf/orbbec_hunter2/actuator/caster.urdf.xacro (robot description, xacro)
@@ -2,18 +2,10 @@
 <robot xmlns:xacro="http://www.ros.org/wiki/xacro">
     <xacro:include filename="$(find ackermancar_description)/urdf/orbbec_hunter2/visual_dir.urdf.xacro"/>
-    <link name="dummy_base">
-    </link>
-    <joint name="dummy_base_joint" type="fixed">
-        <origin xyz="0 0 0" rpy="0 0 0" />
-        <parent link="dummy_base"/>
-        <child link="base_link"/>
-        <axis xyz="0 0 1" />
-    </joint>
     <link name="base_link">
-        <inertial>
+        <!-- <inertial>
             <origin xyz="0.0075625 -0.0046146 -0.13361" rpy="0 0 0" />
             <mass value="75"/>
             <inertia ixx="0.031279" ixy="0" ixz="0" iyy="0.098367" iyz="0" izz="0.11285" />
-        </inertial>
+        </inertial> -->
         <visual>
             <origin xyz="0 0 0" rpy="0 0 0" />
@@ -32,4 +24,12 @@
         </collision>
     </link>
+    <link name="base_footprint">
+    </link>
+    <joint name="base_footprint_joint" type="fixed">
+        <origin rpy="0 0 0" xyz="0 0 0"/>
+        <parent link="base_footprint"/>
+        <child link="base_link"/>
+        <axis xyz="0 0 -0.01"/>
+    </joint>
     <link name="bracket_link">
     </link>

File: ackermancar_description/urdf/orbbec_hunter2/actuator/wheel.urdf.xacro (robot description, xacro)
@@ -45,5 +45,5 @@
             <parent link="front_${prefix}_steering_link" />
             <child link="front_${prefix}_wheel" />
-            <dynamics damping="0.5" friction="0.5"/>
+            <dynamics damping="0.1" friction="0.1"/>
             <axis xyz="0 ${yaxis} 0" />
             <limit effort="1000.0" velocity="100"/>
@@ -55,5 +55,5 @@
             <parent link="base_link" />
             <child link="rear_${prefix}_wheel" />
-            <dynamics damping="0.5" friction="0.5"/>
+            <dynamics damping="0.1" friction="0.1"/>
             <axis xyz="0 ${yaxis} 0" />
             <limit effort="1000.0" velocity="500.0"/>

File: ackermancar_description/urdf/orbbec_hunter2/base/base.urdf.xacro (robot description, xacro)
@@ -1,4 +1,4 @@
 <?xml version="1.0"?>
-<robot name="base" xmlns:xacro="http://www.ros.org/wiki/xacro" >
+<robot name="orbbec_hunter2_base" xmlns:xacro="http://www.ros.org/wiki/xacro" >
     <xacro:include filename="$(find ackermancar_description)/urdf/orbbec_hunter2/actuator/wheel.urdf.xacro"/>
     <xacro:include filename="$(find ackermancar_description)/urdf/orbbec_hunter2/actuator/steer.urdf.xacro"/>

File: ackermancar_description/urdf/orbbec_hunter2/base/hunter_ros2_control.urdf.xacro (robot description, xacro)
@@ -3,8 +3,8 @@
     <xacro:property name="LEFT_WHEEL_KP" value="1000"/>
     <xacro:property name="LEFT_WHEEL_KI" value="10"/>
-    <xacro:property name="LEFT_WHEEL_KD" value="10"/>
+    <xacro:property name="LEFT_WHEEL_KD" value="1"/>
     <xacro:property name="RIGHT_WHEEL_KP" value="1000"/>
     <xacro:property name="RIGHT_WHEEL_KI" value="10"/>
-    <xacro:property name="RIGHT_WHEEL_KD" value="10"/>
+    <xacro:property name="RIGHT_WHEEL_KD" value="1"/>
     <xacro:property name="LINEAR_VELOCITY_KP" value="1000"/>
     <xacro:property name="LINEAR_VELOCITY_KI" value="10"/>
@@ -12,10 +12,10 @@
     <gazebo>
         <plugin name="gazebo_ros_ackermann_drive" filename="libgazebo_ros_ackermann_drive.so">
-            <ros>
-                <namespace>/orbbec_hunter</namespace>
+            <!-- <ros>
+                <namespace>/orbbec_hunter2</namespace>
                 <remapping> cmd_vel:=cmd_vel </remapping>
                 <remapping> odom:=odom </remapping>
                 <remapping> distance:=distance </remapping>
-            </ros>
+            </ros> -->
             <update_rate>50.0</update_rate>
             <!-- wheels -->
@@ -27,5 +27,5 @@
             <left_steering_joint>front_left_steering_joint</left_steering_joint>
             <right_steering_joint>front_right_steering_joint</right_steering_joint>
-            <steering_wheel_joint>steering_joint </steering_wheel_joint>
+            <steering_wheel_joint>steering_joint</steering_wheel_joint>
             <!-- Other parameters remain the same -->
             <max_steer>0.6458</max_steer>
@@ -44,5 +44,5 @@
             <publish_distance>true</publish_distance>
             <odometry_frame>odom</odometry_frame>
-            <robot_base_frame>base_link</robot_base_frame>
+            <robot_base_frame>base_footprint</robot_base_frame>
         </plugin>
     </gazebo>

File: ackermancar_description/urdf/orbbec_hunter2/hunter.urdf (robot description, URDF)
Before this commit: robot Argus_Hunter_2, 18 links, 17 joints
Links:
- removed link dummy_base
- added link base_footprint
- link base_link: geometry collision mesh filename=/home/youngricky/graduation_project_ws/install/ackermancar_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; visual mesh filename=/home/youngricky/graduation_project_ws/install/ackermancar_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
- link depth_camera_link: geometry collision mesh filename=/home/youngricky/graduation_project_ws/install/ackermancar_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; visual mesh filename=/home/youngricky/graduation_project_ws/install/ackermancar_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
- link front_camera_link: geometry collision mesh filename=/home/youngricky/graduation_project_ws/install/ackermancar_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; visual mesh filename=/home/youngricky/graduation_project_ws/install/ackermancar_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
- link front_left_steering_link: geometry collision mesh filename=/home/youngricky/graduation_project_ws/install/ackermancar_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; visual mesh filename=/home/youngricky/graduation_project_ws/install/ackermancar_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
- link front_left_wheel: mass 4.0 -> 20; geometry collision cylinder length=0.14 radius=0.165; visual mesh filename=/home/youngricky/graduation_project_ws/install/ackermancar_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
- link front_right_steering_link: geometry collision mesh filename=/home/youngricky/graduation_project_ws/install/ackermancar_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; visual mesh filename=/home/youngricky/graduation_project_ws/install/ackermancar_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
- link front_right_wheel: mass 4.0 -> 20; geometry collision cylinder length=0.14 radius=0.165; visual mesh filename=/home/youngricky/graduation_project_ws/install/ackermancar_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
- link front_sonar_link: geometry collision mesh filename=/home/youngricky/graduation_project_ws/install/ackermancar_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; visual mesh filename=/home/youngricky/graduation_project_ws/install/ackermancar_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
- link left_camera_link: geometry collision mesh filename=/home/youngricky/graduation_project_ws/install/ackermancar_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; visual mesh filename=/home/youngricky/graduation_project_ws/install/ackermancar_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
- link lidar_link: geometry collision mesh filename=/home/youngricky/graduation_project_ws/install/ackermancar_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; visual mesh filename=/home/youngricky/graduation_project_ws/install/ackermancar_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
- link rear_camera_link: geometry collision mesh filename=/home/youngricky/graduation_project_ws/install/ackermancar_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; visual mesh filename=/home/youngricky/graduation_project_ws/install/ackermancar_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
- link rear_left_wheel: mass 4.0 -> 20; geometry collision cylinder length=0.14 radius=0.165; visual mesh filename=/home/youngricky/graduation_project_ws/install/ackermancar_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
- link rear_right_wheel: mass 4.0 -> 20; geometry collision cylinder length=0.14 radius=0.165; visual mesh filename=/home/youngricky/graduation_project_ws/install/ackermancar_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
- link rear_sonar_link: geometry collision mesh filename=/home/youngricky/graduation_project_ws/install/ackermancar_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; visual mesh filename=/home/youngricky/graduation_project_ws/install/ackermancar_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
- link right_camera_link: geometry collision mesh filename=/home/youngricky/graduation_project_ws/install/ackermancar_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; visual mesh filename=/home/youngricky/graduation_project_ws/install/ackermancar_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
Joints:
- removed joint dummy_base_joint
- added joint base_footprint_joint: type fixed, parent base_link, child base_footprint, origin xyz=0 0 0 rpy=0 0 0, axis 0 0 -1

Commit message: add launch files for mapping

File: ackermancar_description/urdf/orbbec_hunter2/actuator/caster.urdf.xacro (robot description, xacro)
@@ -30,5 +30,5 @@
         <parent link="base_footprint"/>
         <child link="base_link"/>
-        <axis xyz="0 0 -0.01"/>
+        <axis xyz="0 0 0.01"/>
     </joint>
     <link name="bracket_link">

File: ackermancar_description/urdf/orbbec_hunter2/base/hunter_ros2_control_test.urdf.xacro (robot description, xacro)
@@ -61,5 +61,5 @@
     <gazebo>
         <plugin name="gazebo_ros2_control" filename="libgazebo_ros2_control.so">
-            <parameters>$(find ackermancar_description)/config/controller.yaml</parameters>
+            <parameters>$(find ackermancar_description)/params/controller.yaml</parameters>
         </plugin>
     </gazebo>

File: ackermancar_description/urdf/orbbec_hunter2/hunter.urdf (robot description, URDF)
Before this commit: robot orbbec_hunter2, 18 links, 17 joints
Links:
- removed link lidar_link
- added link lidar, mass 0.9; collision mesh filename=package://ackermancar_description/meshes/visual/lidar.STL; visual mesh filename=package://ackermancar_description/meshes/visual/lidar.STL
- link base_link: mass 75 -> None; geometry collision mesh filename=package://ackermancar_description/meshes/visual/chassis_and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; visual mesh filename=package://ackermancar_description/meshes/visual/chassis_and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
- link depth_camera_link: geometry collision mesh filename=package://ackermancar_description/meshes/visual/depth_camer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; visual mesh filename=package://ackermancar_description/meshes/visual/depth_camer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
- link front_camera_link: geometry collision mesh filename=package://ackermancar_description/meshes/visual/camera.STL; visual mesh filename=package://ackermancar_description/meshes/visual/camera.STL
- link front_left_steering_link: geometry collision mesh filename=package://ackermancar_description/meshes/visual/front_left_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; visual mesh filename=package://ackermancar_description/meshes/visual/front_left_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
- link front_left_wheel: geometry collision cylinder length=0.14 radius=0.165; visual mesh filename=package://ackermancar_description/meshes/visual/front_left_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
- link front_right_steering_link: geometry collision mesh filename=package://ackermancar_description/meshes/visual/front_right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; visual mesh filename=package://ackermancar_description/meshes/visual/front_right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
- link front_right_wheel: geometry collision cylinder length=0.14 radius=0.165; visual mesh filename=package://ackermancar_description/meshes/visual/front_right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
- link front_sonar_link: geometry collision mesh filename=package://ackermancar_description/meshes/visual/sonar.STL; visual mesh filename=package://ackermancar_description/meshes/visual/sonar.STL
- link left_camera_link: geometry collision mesh filename=package://ackermancar_description/meshes/visual/camera.STL; visual mesh filename=package://ackermancar_description/meshes/visual/camera.STL
- link rear_camera_link: geometry collision mesh filename=package://ackermancar_description/meshes/visual/camera.STL; visual mesh filename=package://ackermancar_description/meshes/visual/camera.STL
- link rear_left_wheel: geometry collision cylinder length=0.14 radius=0.165; visual mesh filename=package://ackermancar_description/meshes/visual/rear_left_w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
- link rear_right_wheel: geometry collision cylinder length=0.14 radius=0.165; visual mesh filename=package://ackermancar_description/meshes/visual/rear_right_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
- link rear_sonar_link: geometry collision mesh filename=package://ackermancar_description/meshes/visual/sonar.STL; visual mesh filename=package://ackermancar_description/meshes/visual/sonar.STL
- link right_camera_link: geometry collision mesh filename=package://ackermancar_description/meshes/visual/camera.STL; visual mesh filename=package://ackermancar_description/meshes/visual/camera.STL
Joints:
- removed joint lidar_link_joint
- added joint lidar_joint: type fixed, parent bracket_link, child lidar, origin xyz=0.04 0 0.9656 rpy=0 0 0, axis 0 0 -1
- joint base_footprint_joint: axis 0 0 -1 -> 0 0 0.1; child base_footprint -> base_link; parent base_link -> base_footprint

File: ackermancar_description/urdf/orbbec_hunter2/sensor/camera.urdf.xacro (robot description, xacro)
@@ -1,5 +1,5 @@
 <?xml version="1.0"?>
 <robot xmlns:xacro="http://www.ros.org/wiki/xacro">
-    <xacro:include filename="$(find ackermancar_description)/urdf/orbbec_hunter2/visuial_dir.urdf.xacro"/>
+    <xacro:include filename="$(find ackermancar_description)/urdf/orbbec_hunter2/visual_dir.urdf.xacro"/>
     <xacro:macro name="rgb_camera" params="prefix">
         <link name="${prefix}_camera_link">

File: ackermancar_description/urdf/orbbec_hunter2/sensor/imu.urdf.xacro (robot description, xacro)
@@ -1,5 +1,5 @@
 <?xml version="1.0"?>
 <robot xmlns:xacro="http://www.ros.org/wiki/xacro">
-    <xacro:include filename="$(find ackermancar_description)/urdf/orbbec_hunter2/visuial_dir.urdf.xacro"/>
+    <xacro:include filename="$(find ackermancar_description)/urdf/orbbec_hunter2/visual_dir.urdf.xacro"/>
     <!-- imu sensor-->
     <gazebo reference="depth_camera_link">

File: ackermancar_description/urdf/orbbec_hunter2/sensor/laser.urdf.xacro (robot description, xacro)
@@ -1,6 +1,6 @@
 <?xml version="1.0"?>
 <robot xmlns:xacro="http://www.ros.org/wiki/xacro">
-    <xacro:include filename="$(find ackermancar_description)/urdf/orbbec_hunter2/visuial_dir.urdf.xacro"/>
-    <link name="lidar_link">
+    <xacro:include filename="$(find ackermancar_description)/urdf/orbbec_hunter2/visual_dir.urdf.xacro"/>
+    <link name="lidar">
         <inertial>
             <origin xyz="0 0 0.036317" rpy="0 0 0" />
@@ -25,12 +25,12 @@
     </link>
     <!-- LiDAR -->
-    <joint name="lidar_link_joint" type="fixed">
+    <joint name="lidar_joint" type="fixed">
         <origin xyz="0.04 0 0.9656" rpy="0 0 0" />
         <parent link="bracket_link" />
-        <child link="lidar_link" />
+        <child link="lidar" />
         <axis xyz="0 0 -1" />
     </joint>
     <!-- laser sensor -->
-    <gazebo reference="lidar_link">
+    <gazebo reference="lidar">
         <material>Gazebo/Black</material>
         <sensor type="ray" name="rplidar">

File: ackermancar_description/urdf/orbbec_hunter2/sensor/sonar.urdf.xacro (robot description, xacro)
@@ -1,5 +1,5 @@
 <?xml version="1.0"?>
 <robot xmlns:xacro="http://www.ros.org/wiki/xacro">
-<xacro:include filename="$(find ackermancar_description)/urdf/orbbec_hunter2/visuial_dir.urdf.xacro"/>
+<xacro:include filename="$(find ackermancar_description)/urdf/orbbec_hunter2/visual_dir.urdf.xacro"/>
     <xacro:macro name="sonar_link" params="prefix">
         <link name="${prefix}_sonar_link">
