Commit message: add neor_mini car

File: ackermancar_description/urdf/hunter2/actuator/caster.urdf.xacro (robot description, xacro)
@@ -1,5 +1,5 @@
 <?xml version="1.0"?>
 <robot xmlns:xacro="http://www.ros.org/wiki/xacro">
-    <xacro:include filename="$(find ackermancar_description)/urdf/orbbec_hunter2/visual_dir.urdf.xacro"/>
+    <xacro:include filename="$(find ackermancar_description)/urdf/hunter2/visual_dir.urdf.xacro"/>
     <link name="base_link">
         <!-- <inertial>

File: ackermancar_description/urdf/hunter2/actuator/steer.urdf.xacro (robot description, xacro)
@@ -1,5 +1,5 @@
 <?xml version="1.0"?>
 <robot xmlns:xacro="http://www.ros.org/wiki/xacro">
-    <xacro:include filename="$(find ackermancar_description)/urdf/orbbec_hunter2/visual_dir.urdf.xacro"/>
+    <xacro:include filename="$(find ackermancar_description)/urdf/hunter2/visual_dir.urdf.xacro"/>
     <xacro:macro name="steering_link" params="prefix">
         <link name="${prefix}_steering_link">

File: ackermancar_description/urdf/hunter2/actuator/wheel.urdf.xacro (robot description, xacro)
@@ -1,6 +1,5 @@
 <?xml version="1.0"?>
 <robot xmlns:xacro="http://www.ros.org/wiki/xacro">
-    <!-- <xacro:include filename="$(find fishbot_description)/urdf/fishbot/common_inertia.xacro" /> -->
-    <xacro:include filename="$(find ackermancar_description)/urdf/orbbec_hunter2/visual_dir.urdf.xacro" />
+    <xacro:include filename="$(find ackermancar_description)/urdf/hunter2/visual_dir.urdf.xacro" />
     <xacro:property name="wheel_width" value="0.14"/>
     <xacro:property name="wheel_radius" value="0.165"/>
@@ -37,5 +36,5 @@
             <mu2 value="${mu2}"/>
             <kp value="${kp}" />
-            <kd value="${kd}" />
+            <kd value="${kd}" />z
         </gazebo>
     </xacro:macro>

File: ackermancar_description/urdf/hunter2/base/base.urdf.xacro (robot description, xacro)
@@ -1,7 +1,7 @@
 <?xml version="1.0"?>
-<robot name="orbbec_hunter2_base" xmlns:xacro="http://www.ros.org/wiki/xacro" >
-    <xacro:include filename="$(find ackermancar_description)/urdf/orbbec_hunter2/actuator/wheel.urdf.xacro"/>
-    <xacro:include filename="$(find ackermancar_description)/urdf/orbbec_hunter2/actuator/steer.urdf.xacro"/>
-    <xacro:include filename="$(find ackermancar_description)/urdf/orbbec_hunter2/actuator/caster.urdf.xacro"/>
+<robot name="hunter2_base" xmlns:xacro="http://www.ros.org/wiki/xacro" >
+    <xacro:include filename="$(find ackermancar_description)/urdf/hunter2/actuator/wheel.urdf.xacro"/>
+    <xacro:include filename="$(find ackermancar_description)/urdf/hunter2/actuator/steer.urdf.xacro"/>
+    <xacro:include filename="$(find ackermancar_description)/urdf/hunter2/actuator/caster.urdf.xacro"/>
     <xacro:property name="MU1" value="5.0"/>
     <xacro:property name="MU2" value="5.0"/>

File: ackermancar_description/urdf/hunter2/base/hunter_ros2_control.urdf.xacro (robot description, xacro)
@@ -12,10 +12,4 @@
     <gazebo>
         <plugin name="gazebo_ros_ackermann_drive" filename="libgazebo_ros_ackermann_drive.so">
-            <!-- <ros>
-                <namespace>/orbbec_hunter2</namespace>
-                <remapping> cmd_vel:=cmd_vel </remapping>
-                <remapping> odom:=odom </remapping>
-                <remapping> distance:=distance </remapping>
-            </ros> -->
             <update_rate>50.0</update_rate>
             <!-- wheels -->
@@ -55,5 +49,5 @@
             <frame_name>map</frame_name>
             <body_name>base_footprint</body_name>
-            <update_rate>50.0</update_rate>
+            <update_rate>100.0</update_rate>
         </plugin>
     </gazebo>

File: ackermancar_description/urdf/hunter2/base/hunter_ros2_control_test.urdf.xacro (robot description, xacro)
@@ -6,60 +6,29 @@
         </hardware>
         <joint name="front_left_wheel_joint">
-            <command_interface name="velocity">
-                <param name="min">0.0</param>
-                <param name="max">20.0</param>
-            </command_interface>
+            <command_interface name="position"/>
             <state_interface name="position" />
-            <state_interface name="velocity" />
         </joint>
         <joint name="front_right_wheel_joint">
-            <command_interface name="velocity">
-                <param name="min">0.0</param>
-                <param name="max">20.0</param>
-            </command_interface>
+            <command_interface name="position"/>
             <state_interface name="position" />
-            <state_interface name="velocity" />
         </joint>
         <joint name="rear_left_wheel_joint">
-            <command_interface name="velocity">
-                <param name="min">0.0</param>
-                <param name="max">20.0</param>
-            </command_interface>
+            <command_interface name="velocity"/>
             <state_interface name="position" />
             <state_interface name="velocity" />
         </joint>
         <joint name="rear_right_wheel_joint">
-            <command_interface name="velocity">
-                <param name="min">0.0</param>
-                <param name="max">20.0</param>
-            </command_interface>
+            <command_interface name="velocity"/>
             <state_interface name="position" />
             <state_interface name="velocity" />
-        </joint>
-        <joint name="front_left_steering_joint">
-            <command_interface name="position">
-                <param name="min">-1.0</param>
-                <param name="max">1.0</param>
-            </command_interface>
-            <state_interface name="position" />
-        </joint>
-        <joint name="front_right_steering_joint">
-            <command_interface name="position">
-                <param name="min">-1.0</param>
-                <param name="max">1.0</param>
-            </command_interface>
-            <state_interface name="position" />
-        </joint>
-        <joint name="steering_joint">
-            <command_interface name="position">
-                <param name="min">-1.0</param>
-                <param name="max">1.0</param>
-            </command_interface>
-            <state_interface name="position" />
         </joint>
     </ros2_control>
     <gazebo>
         <plugin name="gazebo_ros2_control" filename="libgazebo_ros2_control.so">
-            <parameters>$(find ackermancar_description)/params/controller.yaml</parameters>
+            <parameters>$(find ackermancar_description)/params/hunter2/controller.yaml</parameters>
+            <!-- <ros>
+                <remapping>/hunter2_ackermann_drive_controller/cmd_vel_unstamped:=/cmd_vel</remapping>
+                <remapping>/hunter2_ackermann_drive_controller/odom:=/odom</remapping>
+            </ros> -->
         </plugin>
     </gazebo>

File: ackermancar_description/urdf/hunter2/base/sensor.urdf.xacro (robot description, xacro)
@@ -1,9 +1,9 @@
 <?xml version="1.0"?>
 <robot xmlns:xacro="http://www.ros.org/wiki/xacro">
-    <xacro:include filename="$(find ackermancar_description)/urdf/orbbec_hunter2/visual_dir.urdf.xacro"/>
-    <xacro:include filename="$(find ackermancar_description)/urdf/orbbec_hunter2/sensor/sonar.urdf.xacro"/>
-    <xacro:include filename="$(find ackermancar_description)/urdf/orbbec_hunter2/sensor/camera.urdf.xacro"/>
-    <xacro:include filename="$(find ackermancar_description)/urdf/orbbec_hunter2/sensor/laser.urdf.xacro"/>
-    <xacro:include filename="$(find ackermancar_description)/urdf/orbbec_hunter2/sensor/imu.urdf.xacro"/>
+    <xacro:include filename="$(find ackermancar_description)/urdf/hunter2/visual_dir.urdf.xacro"/>
+    <xacro:include filename="$(find ackermancar_description)/urdf/hunter2/sensor/sonar.urdf.xacro"/>
+    <xacro:include filename="$(find ackermancar_description)/urdf/hunter2/sensor/camera.urdf.xacro"/>
+    <xacro:include filename="$(find ackermancar_description)/urdf/hunter2/sensor/laser.urdf.xacro"/>
+    <xacro:include filename="$(find ackermancar_description)/urdf/hunter2/sensor/imu.urdf.xacro"/>
     <xacro:sonar_link prefix="front"/>
     <xacro:sonar_link prefix="rear"/>

File: ackermancar_description/urdf/hunter2/sensor/camera.urdf.xacro (robot description, xacro)
@@ -1,5 +1,5 @@
 <?xml version="1.0"?>
 <robot xmlns:xacro="http://www.ros.org/wiki/xacro">
-    <xacro:include filename="$(find ackermancar_description)/urdf/orbbec_hunter2/visual_dir.urdf.xacro"/>
+    <xacro:include filename="$(find ackermancar_description)/urdf/hunter2/visual_dir.urdf.xacro"/>
     <xacro:macro name="rgb_camera" params="prefix">
         <link name="${prefix}_camera_link">

File: ackermancar_description/urdf/hunter2/sensor/imu.urdf.xacro (robot description, xacro)
@@ -1,5 +1,5 @@
 <?xml version="1.0"?>
 <robot xmlns:xacro="http://www.ros.org/wiki/xacro">
-    <xacro:include filename="$(find ackermancar_description)/urdf/orbbec_hunter2/visual_dir.urdf.xacro"/>
+    <xacro:include filename="$(find ackermancar_description)/urdf/hunter2/visual_dir.urdf.xacro"/>
     <!-- imu sensor-->
     <gazebo reference="depth_camera_link">

File: ackermancar_description/urdf/hunter2/sensor/laser.urdf.xacro (robot description, xacro)
@@ -1,5 +1,5 @@
 <?xml version="1.0"?>
 <robot xmlns:xacro="http://www.ros.org/wiki/xacro">
-    <xacro:include filename="$(find ackermancar_description)/urdf/orbbec_hunter2/visual_dir.urdf.xacro"/>
+    <xacro:include filename="$(find ackermancar_description)/urdf/hunter2/visual_dir.urdf.xacro"/>
     <link name="lidar">
         <inertial>

File: ackermancar_description/urdf/hunter2/sensor/sonar.urdf.xacro (robot description, xacro)
@@ -1,5 +1,5 @@
 <?xml version="1.0"?>
 <robot xmlns:xacro="http://www.ros.org/wiki/xacro">
-<xacro:include filename="$(find ackermancar_description)/urdf/orbbec_hunter2/visual_dir.urdf.xacro"/>
+<xacro:include filename="$(find ackermancar_description)/urdf/hunter2/visual_dir.urdf.xacro"/>
     <xacro:macro name="sonar_link" params="prefix">
         <link name="${prefix}_sonar_link">
