Commit message: add controller testing tools

File: ackermancar_description/urdf/neor_mini/neor_mini.urdf (robot description, URDF)
Before this commit: robot neor_mini, 12 links, 11 joints
Joints:
- joint front_steer_left_joint: limit lower=-0.69 upper=0.69 effort=4000 velocity=100 -> lower=-0.69 upper=0.69 effort=4000 velocity=5
- joint front_steer_right_joint: limit lower=-0.69 upper=0.69 effort=4000 velocity=100 -> lower=-0.69 upper=0.69 effort=4000 velocity=5
- joint left_rear_joint: limit effort=4000 velocity=100 -> effort=4000 velocity=10
- joint right_rear_joint: limit effort=4000 velocity=100 -> effort=4000 velocity=10
